File: encoder/encoder.kicad_pcb (KiCad board)
At the start: 2 copper layers, 26.5 x 30 mm, 0 parts

Commit message: Made the encoder PCB
Parts:
- added C1: 100nF, Capacitor_SMD:C_0402_1005Metric, F.Cu at (111.9, 111.8)
- added H1: MountingHole_Pad_MP, MountingHole:MountingHole_2.2mm_M2_DIN965_Pad, F.Cu at (114.5, 109.0)
- added H2: MountingHole_Pad_MP, MountingHole:MountingHole_2.2mm_M2_DIN965_Pad, F.Cu at (102.5, 109.0)
- added J1: Conn_01x06_Pin, Connector_PinHeader_1.00mm:PinHeader_1x06_P1.00mm_Vertical, F.Cu at (111.0, 114.0)
- added U1: AS5047P, Package_SO:TSSOP-14_4.4x5mm_P0.65mm, F.Cu at (108.5, 108.9)
Routing:
- net VDD: track 0.00 -> 11.3 mm
- net /MOSI: track 0.00 -> 2.96 mm
- net /MISO: track 0.00 -> 2.71 mm
- net /SCK: track 0.00 -> 2.57 mm
- net /ENC_CS: track 0.00 -> 2.42 mm
- added copper zone on B.Cu, net GND
- added copper zone on F.Cu, net GND
Other:
- board size 26.5 x 30 mm -> 17 x 14.5 mm
- board text added: "AS5047P ENCODER BOGDAN SECZKOWSKI 2026"
