File: encoder/encoder.kicad_sch (KiCad schematic)
At the start: 3 parts, among them J1 Conn_01x06_Pin, U1 AS5047P

Commit message: Made the encoder PCB
Parts:
- added H1, H2: MountingHole_Pad_MP, MountingHole:MountingHole_2.2mm_M2_DIN965_Pad, symbol Mechanical:MountingHole_Pad_MP
Connections:
- net GND: now also H1.MP, H2.MP
