File: servo/Driver.kicad_sch (KiCad schematic)
At the start: 19 parts, among them J7 Conn_01x02_Pin, J9 Conn_01x02_Pin, U4 DRV8263SQVAKRQ1

Commit message: Made the encoder PCB
Parts:
- R16: LCSC Part C242161 -> C482224
Changed lines of the file:
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@@
 			)
 		)
-		(property "LCSC Part" "C242161"
+		(property "LCSC Part" "C482224"
 			(at 189.23 64.77 0)
 			(effects
